File: main.kicad_pcb (KiCad board)
At the start: 2 copper layers, 78 x 47 mm, 59 parts, among them J1 Conn_01x12_Pin, J2 Conn_01x12_Pin, J3 Conn_01x12_Pin, J4 Conn_01x12_Pin, J5 Conn_01x02_Pin

Commit message: update
Parts:
- moved C5-2 40.8 mm to (205.5, 78.7), turned to 90 degrees
- moved C5-1 40.4 mm to (220.5, 78.7), turned to 90 degrees
- moved J5 35.0 mm to (215.1, 77.3), turned to 180 degrees
Other:
- board text added: "N,P,S,D -> GND,POS,SIGNEL,DATA S -> Servo USB -> Webcam C -> Color sensor"
- board text removed: "BB_D1"
- board text removed: "BB_D2"
- board text removed: "BB_N"
- board text removed: "BB_P"
- board text removed: "N,P,S,D -> GND,POS,SIGNEL,DATA S -> Servo BB -> Break beam USB -> Webcam C -> Color sensor"

Commit message: new number
Other:
- board text added: "JLCJLCJLCJLC"
- board text removed: "JLC_BATCH_NUM"
Changed lines of the file:
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@@
 		(tags "connector JST VH vertical")
 		(property "Reference" "J5"
-			(at 1.98 -4.9 360)
+			(at 1.98 -4.9 0)
 			(layer "F.SilkS")
 			(hide yes)
@@
 		)
 		(property "Value" "Conn_01x02_Pin"
-			(at 1.98 6 360)
+			(at 1.98 6 0)
 			(layer "F.Fab")
 			(effects
@@
 		)
 		(fp_text user "${REFERENCE}"
-			(at 1.98 4.1 360)
+			(at 1.98 4.1 0)
 			(layer "F.Fab")
 			(effects
@@
 		)
 	)
-	(gr_text "JLC_BATCH_NUM"
+	(gr_text "JLCJLCJLCJLC"
 		(at 242.55 43.125 0)
 		(layer "B.SilkS")
